File: Hardware/Curios.sch (EAGLE design)
At the start: 0 parts

Commit message: update week 2
Parts:
- added B1: ARDUINO_UNO_R3_SHIELD_ICSP, LinnesLab-Microcontrollers:ARDUINO_UNO_R3_SHIELD_ICSP
- added C1: (no value), LinnesLab-Passives:CAPACITOR0603
- added IC1: AD623N, LinnesLab-AnalogIC:AD623N
- added OP1: (no value), LinnesLab-AnalogIC:OP-DUALR
- added R1: (no value), LinnesLab-Passives:RESISTOR0603
Connections:
- new net 5V: B1.5V
- new net GND: B1.GND@2
- new net N$10: IC1.OUT
- new net N$11: B1.A0
- new net N$3: IC1.+
- new net N$4: IC1.RG@1
- new net N$5: IC1.RG@2
- new net N$6: IC1.-
- new net N$7: IC1.+V
- new net N$8: IC1.REF
- new net N$9: IC1.-V
