File: Hardware/Curios.sch (EAGLE design)
At the start: 5 parts, among them IC1 AD623N

Commit message: Week6 update
Parts:
- removed C1: (no value), LinnesLab-Passives:CAPACITOR0603
- added CF: 3.3nF, LinnesLab-Passives:CAPACITOR0603
- added CIN1, CIN2: 0.47uF, LinnesLab-Passives:CAPACITOR0603
- added R2, R3: 10k, LinnesLab-Passives:RESISTOR0603
- added RF: 47k, LinnesLab-Passives:RESISTOR0603
- added RIN: 2.2k, LinnesLab-Passives:RESISTOR0603
- R1: value (none) -> 10k
Connections:
- net N$11 renamed OUTPUT
- removed net N$8: IC1.REF
- removed net N$9: IC1.-V
- new net 3.3V: B1.3.3V, R1.2
- new net N$1: CIN1.1, CIN2.1, RIN.2
- new net N$2: OP1A.+IN, OP1B.-IN, OP1B.OUT
- net 5V: now also OP1P.V+
- net GND: now also OP1P.V-, R2.1
- net N$10: now also CF.2, OP1A.OUT, RF.2; no longer IC1.OUT
- net N$3: now also OP1B.+IN, R1.1, R2.2; no longer IC1.+
- net N$4: now also IC1.OUT, RIN.1; no longer IC1.RG@1
- net N$5: now also IC1.RG@1, R3.1; no longer IC1.RG@2
- net N$6: now also CF.1, CIN1.2, CIN2.2, OP1A.-IN, RF.1; no longer IC1.-
- net N$7: now also IC1.RG@2, R3.2; no longer IC1.+V
Other:
- moved on the sheet: IC1, OP1A, OP1B, OP1P, R1

Commit message: Week 6 update
Parts:
- added CSAFE: 3.3nF, LinnesLab-Passives:CAPACITOR0603
- added J1: (no value), LinnesLab-Connectors:AUDIO_JACK_TRRSSMD_RA
- R3: value 10k -> 22k
Connections:
- removed net 5V: B1.5V, OP1P.V+
- removed net N$10: CF.2, OP1A.OUT, RF.2
- new net N$8: IC1.-, J1.TIP
- new net VREF: IC1.REF, OP1A.+IN, OP1B.-IN, OP1B.OUT
- net 3.3V: now also CSAFE.2, IC1.+V, OP1P.V+
- net GND: now also B1.GND, B1.GND@0, B1.GND@1, CSAFE.1, IC1.-V, J1.RING2, J1.SLEEVE
- net N$2: now also IC1.+, J1.RING1; no longer OP1A.+IN, OP1B.-IN, OP1B.OUT
- net OUTPUT: now also CF.2, OP1A.OUT, RF.2
Other:
- moved on the sheet: B1
Changed lines of the file:
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@@
 <part name="B1" library="LinnesLab-Microcontrollers" deviceset="ARDUINO_UNO_R3_SHIELD_ICSP" device=""/>
 <part name="IC1" library="LinnesLab-AnalogIC" deviceset="AD623" device="N" package3d_urn="urn:adsk.eagle:package:16409/2"/>
-<part name="SUPPLY1" library="LinnesLab-Symbols" deviceset="5V" device=""/>
 <part name="RF" library="LinnesLab-Passives" deviceset="RESISTOR" device="0603" package3d_urn="urn:adsk.eagle:package:15661944/2" value="47k"/>
 <part name="CF" library="LinnesLab-Passives" deviceset="CAPACITOR" device="0603" package3d_urn="urn:adsk.eagle:package:15661989/2" value="3.3nF"/>
@@
 <part name="R2" library="LinnesLab-Passives" deviceset="RESISTOR" device="0603" package3d_urn="urn:adsk.eagle:package:15661944/2" value="10k"/>
 <part name="SUPPLY2" library="LinnesLab-Symbols" deviceset="3.3V" device=""/>
-<part name="R3" library="LinnesLab-Passives" deviceset="RESISTOR" device="0603" package3d_urn="urn:adsk.eagle:package:15661944/2" value="10k"/>
+<part name="R3" library="LinnesLab-Passives" deviceset="RESISTOR" device="0603" package3d_urn="urn:adsk.eagle:package:15661944/2" value="22k"/>
+<part name="J1" library="LinnesLab-Connectors" deviceset="AUDIO_JACK_TRRS" device="SMD_RA" package3d_urn="urn:adsk.eagle:package:18169774/2"/>
+<part name="CSAFE" library="LinnesLab-Passives" deviceset="CAPACITOR" device="0603" package3d_urn="urn:adsk.eagle:package:15661989/2" value="3.3nF"/>
 </parts>
 <sheets>
@@
 </plain>
 <instances>
-<instance part="B1" gate="G$1" x="15.24" y="53.34" smashed="yes">
-<attribute name="NAME" x="5.588" y="84.582" size="1.778" layer="95" font="vector"/>
-<attribute name="VALUE" x="5.08" y="22.606" size="1.778" layer="96" font="vector" align="top-left"/>
+<instance part="B1" gate="G$1" x="2.54" y="53.34" smashed="yes">
+<attribute name="NAME" x="-7.112" y="84.582" size="1.778" layer="95" font="vector"/>
+<attribute name="VALUE" x="-7.62" y="22.606" size="1.778" layer="96" font="vector" align="top-left"/>
 </instance>
 <instance part="IC1" gate="G$1" x="53.34" y="58.42" smashed="yes">
@@
 <attribute name="VALUE" x="64.77" y="53.34" size="1.778" layer="96"/>
 </instance>
-<instance part="SUPPLY1" gate="G$1" x="63.5" y="20.32" smashed="yes">
-<attribute name="VALUE" x="63.5" y="23.114" size="1.778" layer="96" align="bottom-center"/>
-</instance>
 <instance part="RF" gate="G$1" x="124.46" y="58.42" smashed="yes">
 <attribute name="NAME" x="120.65" y="59.9186" size="1.778" layer="95"/>
@@
 <attribute name="NAME" x="42.1386" y="62.23" size="1.778" layer="95" rot="R270"/>
 <attribute name="VALUE" x="37.338" y="62.23" size="1.778" layer="96" rot="R270"/>
+</instance>
+<instance part="J1" gate="G$1" x="25.4" y="58.42" smashed="yes">
+<attribute name="NAME" x="20.32" y="64.008" size="1.778" layer="95"/>
+<attribute name="VALUE" x="20.32" y="50.8" size="1.778" layer="96"/>
+</instance>
+<instance part="CSAFE" gate="G$1" x="83.82" y="45.72" smashed="yes" rot="R180">
+<attribute name="NAME" x="82.296" y="42.799" size="1.778" layer="95" rot="R180"/>
+<attribute name="VALUE" x="84.836" y="47.879" size="1.778" layer="96" rot="R180"/>
 </instance>
 </instances>
@@
 </busses>
 <nets>
-<net name="5V" class="0">
-<segment>
-<pinref part="B1" gate="G$1" pin="5V"/>
-<wire x1="2.54" y1="55.88" x2="0" y2="55.88" width="0.1524" layer="91"/>
-<label x="-2.54" y="55.88" size="1.778" layer="95"/>
-</segment>
-<segment>
-<pinref part="OP1" gate="P" pin="V+"/>
-<wire x1="91.44" y1="50.8" x2="91.44" y2="53.34" width="0.1524" layer="91"/>
-<label x="91.44" y="53.34" size="1.778" layer="95"/>
-</segment>
-</net>
 <net name="GND" class="0">
 <segment>
 <pinref part="B1" gate="G$1" pin="GND@2"/>
-<wire x1="2.54" y1="48.26" x2="0" y2="48.26" width="0.1524" layer="91"/>
-<label x="-2.54" y="48.26" size="1.778" layer="95"/>
+<wire x1="-10.16" y1="48.26" x2="-12.7" y2="48.26" width="0.1524" layer="91"/>
+<label x="-15.24" y="48.26" size="1.778" layer="95"/>
 </segment>
 <segment>
@@
 <wire x1="91.44" y1="35.56" x2="91.44" y2="33.02" width="0.1524" layer="91"/>
 <label x="91.44" y="33.02" size="1.778" layer="95"/>
+<pinref part="CSAFE" gate="G$1" pin="1"/>
+<wire x1="83.82" y1="40.64" x2="83.82" y2="35.56" width="0.1524" layer="91"/>
+<wire x1="83.82" y1="35.56" x2="91.44" y2="35.56" width="0.1524" layer="91"/>
+<junction x="91.44" y="35.56"/>
 </segment>
 <segment>
 <pinref part="R2" gate="G$1" pin="1"/>
 <wire x1="83.82" y1="91.44" x2="81.28" y2="91.44" width="0.1524" layer="91"/>
-<label x="78.74" y="93.98" size="1.778" layer="95"/>
+<label x="81.28" y="91.44" size="1.778" layer="95"/>
+</segment>
+<segment>
+<pinref part="IC1" gate="G$1" pin="-V"/>
+<wire x1="53.34" y1="43.18" x2="53.34" y2="40.64" width="0.1524" layer="91"/>
+<label x="53.34" y="38.1" size="1.778" layer="95"/>
+</segment>
+<segment>
+<pinref part="B1" gate="G$1" pin="GND@1"/>
+<wire x1="-10.16" y1="45.72" x2="-12.7" y2="45.72" width="0.1524" layer="91"/>
+<label x="-15.24" y="45.72" size="1.778" layer="95"/>
+</segment>
+<segment>
+<pinref part="B1" gate="G$1" pin="GND@0"/>
+<wire x1="-10.16" y1="43.18" x2="-12.7" y2="43.18" width="0.1524" layer="91"/>
+<label x="-15.24" y="43.18" size="1.778" layer="95"/>
+</segment>
+<segment>
+<pinref part="B1" gate="G$1" pin="GND"/>
+<wire x1="-10.16" y1="25.4" x2="-12.7" y2="25.4" width="0.1524" layer="91"/>
+<label x="-15.24" y="25.4" size="1.778" layer="95"/>
+</segment>
+<segment>
+<pinref part="J1" gate="G$1" pin="SLEEVE"/>
+<wire x1="30.48" y1="63.5" x2="30.48" y2="68.58" width="0.1524" layer="91"/>
+<label x="30.48" y="68.58" size="1.778" layer="95"/>
+</segment>
+<segment>
+<pinref part="J1" gate="G$1" pin="RING2"/>
+<wire x1="30.48" y1="53.34" x2="30.48" y2="48.26" width="0.1524" layer="91"/>
+<label x="30.48" y="48.26" size="1.778" layer="95"/>
 </segment>
 </net>
@@
 <segment>
 <pinref part="B1" gate="G$1" pin="A0"/>
-<wire x1="2.54" y1="81.28" x2="0" y2="81.28" width="0.1524" layer="91"/>
-<label x="-2.54" y="83.82" size="1.778" layer="95"/>
-</segment>
-</net>
-<net name="N$10" class="0">
+<wire x1="-10.16" y1="81.28" x2="-12.7" y2="81.28" width="0.1524" layer="91"/>
+<label x="-15.24" y="83.82" size="1.778" layer="95"/>
+</segment>
 <segment>
 <pinref part="CF" gate="G$1" pin="2"/>
@@
 <pinref part="OP1" gate="A" pin="OUT"/>
 <wire x1="139.7" y1="73.66" x2="144.78" y2="73.66" width="0.1524" layer="91"/>
+<wire x1="144.78" y1="73.66" x2="147.32" y2="73.66" width="0.1524" layer="91"/>
+<junction x="144.78" y="73.66"/>
+<label x="149.86" y="73.66" size="1.778" layer="95"/>
 </segment>
 </net>
@@
 </segment>
 </net>
-<net name="N$2" class="0">
+<net name="VREF" class="0">
 <segment>
 <pinref part="OP1" gate="A" pin="+IN"/>
@@
 <wire x1="104.14" y1="86.36" x2="119.38" y2="86.36" width="0.1524" layer="91"/>
 <junction x="119.38" y="86.36"/>
+<wire x1="119.38" y1="93.98" x2="121.92" y2="93.98" width="0.1524" layer="91"/>
+<junction x="119.38" y="93.98"/>
+<label x="124.46" y="93.98" size="1.778" layer="95"/>
+</segment>
+<segment>
+<pinref part="IC1" gate="G$1" pin="REF"/>
+<wire x1="58.42" y1="48.26" x2="58.42" y2="45.72" width="0.1524" layer="91"/>
+<label x="58.42" y="45.72" size="1.778" layer="95"/>
 </segment>
 </net>
@@
 <segment>
 <pinref part="B1" gate="G$1" pin="3.3V"/>
-<wire x1="2.54" y1="53.34" x2="0" y2="53.34" width="0.1524" layer="91"/>
-<label x="-2.54" y="53.34" size="1.778" layer="95"/>
+<wire x1="-10.16" y1="53.34" x2="-12.7" y2="53.34" width="0.1524" layer="91"/>
+<label x="-15.24" y="53.34" size="1.778" layer="95"/>
+</segment>
+<segment>
+<pinref part="IC1" gate="G$1" pin="+V"/>
+<wire x1="53.34" y1="73.66" x2="53.34" y2="76.2" width="0.1524" layer="91"/>
+<label x="53.34" y="76.2" size="1.778" layer="95"/>
 </segment>
 <segment>
 <pinref part="R1" gate="G$1" pin="2"/>
 <wire x1="83.82" y1="101.6" x2="81.28" y2="101.6" width="0.1524" layer="91"/>
-<label x="78.74" y="104.14" size="1.778" layer="95"/>
+<label x="81.28" y="104.14" size="1.778" layer="95"/>
+</segment>
+<segment>
+<pinref part="OP1" gate="P" pin="V+"/>
+<wire x1="91.44" y1="50.8" x2="91.44" y2="53.34" width="0.1524" layer="91"/>
+<label x="93.98" y="53.34" size="1.778" layer="95"/>
+<pinref part="CSAFE" gate="G$1" pin="2"/>
+<wire x1="83.82" y1="48.26" x2="83.82" y2="50.8" width="0.1524" layer="91"/>
+<wire x1="83.82" y1="50.8" x2="91.44" y2="50.8" width="0.1524" layer="91"/>
+<junction x="91.44" y="50.8"/>
 </segment>
 </net>
@@
 </segment>
 </net>
+<net name="N$8" class="0">
+<segment>
+<pinref part="IC1" gate="G$1" pin="-"/>
+<pinref part="J1" gate="G$1" pin="TIP"/>
+<wire x1="30.48" y1="55.88" x2="35.56" y2="55.88" width="0.1524" layer="91"/>
+<wire x1="35.56" y1="55.88" x2="35.56" y2="48.26" width="0.1524" layer="91"/>
+<wire x1="35.56" y1="48.26" x2="45.72" y2="48.26" width="0.1524" layer="91"/>
+</segment>
+</net>
+<net name="N$2" class="0">
+<segment>
+<pinref part="J1" gate="G$1" pin="RING1"/>
+<wire x1="30.48" y1="60.96" x2="35.56" y2="60.96" width="0.1524" layer="91"/>
+<wire x1="35.56" y1="60.96" x2="35.56" y2="68.58" width="0.1524" layer="91"/>
+<pinref part="IC1" gate="G$1" pin="+"/>
+<wire x1="35.56" y1="68.58" x2="45.72" y2="68.58" width="0.1524" layer="91"/>
+</segment>
+</net>
