File: Hardware/Curios.brd (EAGLE design)
At the start: 160 x 100 mm, 0 parts

Commit message: update week 2
Parts:
- added B1: ARDUINO_UNO_R3_SHIELD_ICSP, LinnesLab-Microcontrollers:UNO_R3_SHIELD_ICSP
- added C1: (no value), LinnesLab-Passives:C0603
- added IC1: AD623N, LinnesLab-AnalogIC:DIL08
- added OP1: (no value), LinnesLab-AnalogIC:SO8
- added R1: (no value), LinnesLab-Passives:R0603
Connections:
- new net 5V: B1.5V
- new net GND: B1.GND@2
- new net N$10: IC1.6
- new net N$11: B1.A0
- new net N$3: IC1.3
- new net N$4: IC1.1
- new net N$5: IC1.8
- new net N$6: IC1.2
- new net N$7: IC1.7
- new net N$8: IC1.5
- new net N$9: IC1.4
- new net V+: OP1.8
- new net V-: OP1.4
