File: Hardware/Curios.brd (EAGLE design)
At the start: 160 x 100 mm, 5 parts, among them IC1 AD623N

Commit message: Week6 update
Parts:
- added CIN1, CIN2: 0.47uF, LinnesLab-Passives:C0603
- added R2, R3: 10k, LinnesLab-Passives:R0603
- added RF: 47k, LinnesLab-Passives:R0603
- added RIN: 2.2k, LinnesLab-Passives:R0603
- CF: value (none) -> 3.3nF
- R1: value (none) -> 10k
- moved R1 33.0 mm to (-50.8, -44.5)
- renumbered C1 to CF
Connections:
- net N$11 renamed OUTPUT
- net N$7 renamed +V
- net N$9 renamed -V
- removed net N$8: IC1.5
- removed net V+: OP1.8
- removed net V-: OP1.4
- new net 3.3V: B1.3.3V, R1.2
- new net N$1: CIN1.1, CIN2.1, RIN.2
- new net N$2: OP1.3, OP1.6, OP1.7
- new net N$7: IC1.8, R3.2
- net 5V: now also OP1.8
- net GND: now also OP1.4, R2.1
- net N$10: now also CF.2, OP1.1, RF.2; no longer IC1.6
- net N$3: now also OP1.5, R1.1, R2.2; no longer IC1.3
- net N$4: now also IC1.6, RIN.1; no longer IC1.1
- net N$5: now also IC1.1, R3.1; no longer IC1.8
- net N$6: now also CF.1, CIN1.2, CIN2.2, OP1.2, RF.1; no longer IC1.2
Changed lines of the file:
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@@
 <attribute name="VALUE" x="-49.276" y="-5.715" size="1.27" layer="27" ratio="10"/>
 </element>
-<element name="R1" library="LinnesLab-Passives" package="R0603" package3d_urn="urn:adsk.eagle:package:15661944/2" value="" x="-50.8" y="-11.43" smashed="yes">
+<element name="RF" library="LinnesLab-Passives" package="R0603" package3d_urn="urn:adsk.eagle:package:15661944/2" value="47k" x="-50.8" y="-11.43" smashed="yes">
 <attribute name="NAME" x="-51.435" y="-10.795" size="0.7112" layer="25"/>
 <attribute name="VALUE" x="-51.435" y="-13.335" size="0.7112" layer="27"/>
 </element>
-<element name="C1" library="LinnesLab-Passives" package="C0603" package3d_urn="urn:adsk.eagle:package:15661989/2" value="" x="-50.8" y="-15.24" smashed="yes">
+<element name="CF" library="LinnesLab-Passives" package="C0603" package3d_urn="urn:adsk.eagle:package:15661989/2" value="3.3nF" x="-50.8" y="-15.24" smashed="yes">
 <attribute name="NAME" x="-51.435" y="-14.605" size="0.7112" layer="25"/>
 <attribute name="VALUE" x="-51.435" y="-17.145" size="0.7112" layer="27"/>
@@
 <attribute name="VALUE" x="-43.815" y="-24.765" size="1.27" layer="27" rot="R90"/>
 </element>
+<element name="RIN" library="LinnesLab-Passives" package="R0603" package3d_urn="urn:adsk.eagle:package:15661944/2" value="2.2k" x="-50.8" y="-29.21" smashed="yes">
+<attribute name="NAME" x="-51.435" y="-28.575" size="0.7112" layer="25"/>
+<attribute name="VALUE" x="-51.435" y="-31.115" size="0.7112" layer="27"/>
+</element>
+<element name="CIN2" library="LinnesLab-Passives" package="C0603" package3d_urn="urn:adsk.eagle:package:15661989/2" value="0.47uF" x="-50.8" y="-34.29" smashed="yes">
+<attribute name="NAME" x="-51.435" y="-33.655" size="0.7112" layer="25"/>
+<attribute name="VALUE" x="-51.435" y="-36.195" size="0.7112" layer="27"/>
+</element>
+<element name="CIN1" library="LinnesLab-Passives" package="C0603" package3d_urn="urn:adsk.eagle:package:15661989/2" value="0.47uF" x="-50.8" y="-39.37" smashed="yes">
+<attribute name="NAME" x="-51.435" y="-38.735" size="0.7112" layer="25"/>
+<attribute name="VALUE" x="-51.435" y="-41.275" size="0.7112" layer="27"/>
+</element>
+<element name="R1" library="LinnesLab-Passives" package="R0603" package3d_urn="urn:adsk.eagle:package:15661944/2" value="10k" x="-50.8" y="-44.45" smashed="yes">
+<attribute name="NAME" x="-51.435" y="-43.815" size="0.7112" layer="25"/>
+<attribute name="VALUE" x="-51.435" y="-46.355" size="0.7112" layer="27"/>
+</element>
+<element name="R2" library="LinnesLab-Passives" package="R0603" package3d_urn="urn:adsk.eagle:package:15661944/2" value="10k" x="-50.8" y="-49.53" smashed="yes">
+<attribute name="NAME" x="-51.435" y="-48.895" size="0.7112" layer="25"/>
+<attribute name="VALUE" x="-51.435" y="-51.435" size="0.7112" layer="27"/>
+</element>
+<element name="R3" library="LinnesLab-Passives" package="R0603" package3d_urn="urn:adsk.eagle:package:15661944/2" value="10k" x="-50.8" y="-54.61" smashed="yes">
+<attribute name="NAME" x="-51.435" y="-53.975" size="0.7112" layer="25"/>
+<attribute name="VALUE" x="-51.435" y="-56.515" size="0.7112" layer="27"/>
+</element>
 </elements>
 <signals>
-<signal name="V+">
-<contactref element="OP1" pad="8"/>
-</signal>
-<signal name="V-">
-<contactref element="OP1" pad="4"/>
-</signal>
 <signal name="5V">
 <contactref element="B1" pad="5V"/>
+<contactref element="OP1" pad="8"/>
+<wire x1="-2.54" y1="45.72" x2="-50.165" y2="-20.26" width="0" layer="19" extent="1-1"/>
 </signal>
 <signal name="GND">
 <contactref element="B1" pad="GND@2"/>
+<contactref element="OP1" pad="4"/>
+<contactref element="R2" pad="1"/>
+<wire x1="-46.355" y1="-25.46" x2="-51.65" y2="-49.53" width="0" layer="19" extent="1-1"/>
+<wire x1="-50.8" y1="34.036" x2="-46.355" y2="-25.46" width="0" layer="19" extent="1-1"/>
+</signal>
+<signal name="N$6">
+<contactref element="RF" pad="1"/>
+<contactref element="CF" pad="1"/>
+<contactref element="CIN2" pad="2"/>
+<contactref element="CIN1" pad="2"/>
+<contactref element="OP1" pad="2"/>
+<wire x1="-49.95" y1="-34.29" x2="-49.95" y2="-39.37" width="0" layer="19" extent="1-1"/>
+<wire x1="-48.895" y1="-25.46" x2="-49.95" y2="-34.29" width="0" layer="19" extent="1-1"/>
+<wire x1="-51.65" y1="-15.24" x2="-48.895" y2="-25.46" width="0" layer="19" extent="1-1"/>
+<wire x1="-51.65" y1="-11.43" x2="-51.65" y2="-15.24" width="0" layer="19" extent="1-1"/>
+</signal>
+<signal name="OUTPUT">
+<contactref element="B1" pad="A0"/>
+</signal>
+<signal name="N$10">
+<contactref element="CF" pad="2"/>
+<contactref element="RF" pad="2"/>
+<contactref element="OP1" pad="1"/>
+<wire x1="-49.95" y1="-15.24" x2="-50.165" y2="-25.46" width="0" layer="19" extent="1-1"/>
+<wire x1="-49.95" y1="-11.43" x2="-49.95" y2="-15.24" width="0" layer="19" extent="1-1"/>
+</signal>
+<signal name="N$1">
+<contactref element="RIN" pad="2"/>
+<contactref element="CIN2" pad="1"/>
+<contactref element="CIN1" pad="1"/>
+<wire x1="-51.65" y1="-34.29" x2="-51.65" y2="-39.37" width="0" layer="19" extent="1-1"/>
+<wire x1="-49.95" y1="-29.21" x2="-51.65" y2="-34.29" width="0" layer="19" extent="1-1"/>
+</signal>
+<signal name="-V">
+<contactref element="IC1" pad="4"/>
+</signal>
+<signal name="+V">
+<contactref element="IC1" pad="7"/>
+</signal>
+<signal name="N$2">
+<contactref element="OP1" pad="3"/>
+<contactref element="OP1" pad="7"/>
+<contactref element="OP1" pad="6"/>
+<wire x1="-47.625" y1="-20.26" x2="-47.625" y2="-25.46" width="0" layer="19" extent="1-1"/>
+<wire x1="-48.895" y1="-20.26" x2="-47.625" y2="-20.26" width="0" layer="19" extent="1-1"/>
+</signal>
+<signal name="3.3V">
+<contactref element="B1" pad="3.3V"/>
+<contactref element="R1" pad="2"/>
+<wire x1="-2.54" y1="43.18" x2="-49.95" y2="-44.45" width="0" layer="19" extent="1-1"/>
 </signal>
 <signal name="N$3">
-<contactref element="IC1" pad="3"/>
+<contactref element="R1" pad="1"/>
+<contactref element="R2" pad="2"/>
+<contactref element="OP1" pad="5"/>
+<wire x1="-51.65" y1="-44.45" x2="-49.95" y2="-49.53" width="0" layer="19" extent="1-1"/>
+<wire x1="-46.355" y1="-20.26" x2="-51.65" y2="-44.45" width="0" layer="19" extent="1-1"/>
 </signal>
 <signal name="N$4">
-<contactref element="IC1" pad="1"/>
+<contactref element="IC1" pad="6"/>
+<contactref element="RIN" pad="1"/>
+<wire x1="-44.45" y1="-1.27" x2="-51.65" y2="-29.21" width="0" layer="19" extent="1-1"/>
 </signal>
 <signal name="N$5">
-<contactref element="IC1" pad="8"/>
-</signal>
-<signal name="N$6">
-<contactref element="IC1" pad="2"/>
+<contactref element="R3" pad="1"/>
+<contactref element="IC1" pad="1"/>
+<wire x1="-49.53" y1="-8.89" x2="-51.65" y2="-54.61" width="0" layer="19" extent="1-1"/>
 </signal>
 <signal name="N$7">
-<contactref element="IC1" pad="7"/>
-</signal>
-<signal name="N$8">
-<contactref element="IC1" pad="5"/>
-</signal>
-<signal name="N$9">
-<contactref element="IC1" pad="4"/>
-</signal>
-<signal name="N$10">
-<contactref element="IC1" pad="6"/>
-</signal>
-<signal name="N$11">
-<contactref element="B1" pad="A0"/>
+<contactref element="R3" pad="2"/>
+<contactref element="IC1" pad="8"/>
+<wire x1="-49.53" y1="-1.27" x2="-49.95" y2="-54.61" width="0" layer="19" extent="1-1"/>
 </signal>
 </signals>

Commit message: Week 6 update
Parts:
- added CSAFE: 3.3nF, LinnesLab-Passives:C0603
- added J1: (no value), LinnesLab-Connectors:AUDIO_JACK_3.5MM_TRRS_SMD_RA
- R3: value 10k -> 22k
- moved R3 149.6 mm to (45.7, 59.7), turned to 270 degrees
- moved RF 112.4 mm to (41.9, 52.1), turned to 90 degrees
- moved CIN1 111.5 mm to (16.5, 49.5)
- moved CF 110.5 mm to (36.8, 52.1), turned to 90 degrees
- moved R2 109.7 mm to (15.2, 38.1), turned to 270 degrees
- moved R1 109.7 mm to (22.9, 36.8), turned to 270 degrees
- moved CIN2 105.5 mm to (16.5, 47.0)
- moved IC1 104.9 mm to (36.8, 59.7), turned to 180 degrees
- moved OP1 101.6 mm to (26.7, 45.7), turned to 270 degrees
- moved RIN 99.8 mm to (16.5, 44.5), turned to 180 degrees
- moved B1 53.6 mm to (26.7, 52.1)
Connections:
- removed net +V: IC1.7
- removed net -V: IC1.4
- removed net 5V: B1.5V, OP1.8
- removed net N$10: CF.2, OP1.1, RF.2
- new net N$8: IC1.2, J1.LEFT
- new net VREF: IC1.5, OP1.3, OP1.6, OP1.7
- net 3.3V: now also CSAFE.2, IC1.7, OP1.8
- net GND: now also B1.GND@0, B1.GND@1, B1.GND_ICSP, CSAFE.1, IC1.4, J1.GND, J1.GND/MIC
- net N$2: now also IC1.3, J1.RIGHT; no longer OP1.3, OP1.6, OP1.7
- net OUTPUT: now also CF.2, OP1.1, RF.2
Routing:
- net GND: track 0.00 -> 143.1 mm
- net 3.3V: track 0.00 -> 51.0 mm, vias 0 -> 1
- net N$6: track 0.00 -> 39.0 mm, vias 0 -> 2
- net N$4: track 0.00 -> 38.8 mm
- net OUTPUT: track 0.00 -> 34.3 mm
- net VREF: track 0.00 -> 19.1 mm, vias 0 -> 1
- net N$3: track 0.00 -> 16.7 mm
- net N$2: track 0.00 -> 14.0 mm
- net N$8: track 0.00 -> 9.39 mm
- net N$7: track 0.00 -> 6.31 mm
- net N$5: track 0.00 -> 6.31 mm
- net N$1: track 0.00 -> 5.67 mm
Other:
- board size 160 x 100 mm -> 53.3 x 59.7 mm

Commit message: Week7
Parts:
- moved R3 1.27 mm to (44.5, 59.7)
Routing:
- net GND: track 143.1 -> 137.5 mm
- net N$6: track 39.0 -> 43.6 mm
- net 3.3V: track 51.0 -> 54.7 mm
- net OUTPUT: track 34.3 -> 36.1 mm
- net N$7: track 6.31 -> 5.04 mm
- net N$5: track 6.31 -> 5.04 mm
- net N$4: track 38.8 -> 39.6 mm
Changed lines of the file:
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@@
 <attribute name="VALUE" x="13.335" y="38.735" size="0.7112" layer="27" rot="R270"/>
 </element>
-<element name="R3" library="LinnesLab-Passives" package="R0603" package3d_urn="urn:adsk.eagle:package:15661944/2" value="22k" x="45.72" y="59.69" smashed="yes" rot="R270">
-<attribute name="NAME" x="46.355" y="60.325" size="0.7112" layer="25" rot="R270"/>
-<attribute name="VALUE" x="43.815" y="60.325" size="0.7112" layer="27" rot="R270"/>
+<element name="R3" library="LinnesLab-Passives" package="R0603" package3d_urn="urn:adsk.eagle:package:15661944/2" value="22k" x="44.45" y="59.69" smashed="yes" rot="R270">
+<attribute name="NAME" x="45.085" y="60.325" size="0.7112" layer="25" rot="R270"/>
+<attribute name="VALUE" x="42.545" y="60.325" size="0.7112" layer="27" rot="R270"/>
 </element>
 <element name="RF" library="LinnesLab-Passives" package="R0603" package3d_urn="urn:adsk.eagle:package:15661944/2" value="47k" x="41.91" y="52.07" smashed="yes" rot="R90">
@@
 <wire x1="34.85" y1="75.64" x2="34.85" y2="69.98" width="0.1524" layer="1"/>
 <wire x1="31.60999375" y1="78.88000625" x2="34.85" y2="75.64" width="0.1524" layer="1"/>
-<wire x1="33.02" y1="63.5" x2="34.3027625" y2="63.5" width="0.1524" layer="16"/>
-<wire x1="34.3027625" y1="63.5" x2="35.1917625" y2="64.389" width="0.1524" layer="16"/>
-<wire x1="35.1917625" y1="64.389" x2="42.291" y2="64.389" width="0.1524" layer="16"/>
-<wire x1="42.291" y1="64.389" x2="50.8" y2="55.88" width="0.1524" layer="16"/>
 <wire x1="50.8" y1="55.88" x2="50.8" y2="53.34" width="0.1524" layer="16"/>
-<wire x1="41.8972375" y1="53.34" x2="50.8" y2="53.34" width="0.1524" layer="16"/>
-<wire x1="38.4682375" y1="56.769" x2="41.8972375" y2="53.34" width="0.1524" layer="16"/>
-<wire x1="2.54" y1="39.116" x2="20.193" y2="56.769" width="0.1524" layer="16"/>
-<wire x1="20.193" y1="56.769" x2="38.4682375" y2="56.769" width="0.1524" layer="16"/>
 <wire x1="46.99" y1="51.65" x2="48.68" y2="53.34" width="0.1524" layer="1"/>
 <wire x1="48.68" y1="53.34" x2="50.8" y2="53.34" width="0.1524" layer="1"/>
@@
 <wire x1="2.54" y1="39.116" x2="15.074" y2="39.116" width="0.1524" layer="1"/>
 <wire x1="15.074" y1="39.116" x2="15.24" y2="38.95" width="0.1524" layer="1"/>
+<wire x1="41.91" y1="64.77" x2="34.29" y2="64.77" width="0.1524" layer="16"/>
+<wire x1="34.29" y1="64.77" x2="33.02" y2="63.5" width="0.1524" layer="16"/>
+<wire x1="50.8" y1="55.88" x2="41.91" y2="64.77" width="0.1524" layer="16"/>
+<wire x1="7.62" y1="58.42" x2="7.62" y2="40.64" width="0.1524" layer="16"/>
+<wire x1="7.62" y1="40.64" x2="6.096" y2="39.116" width="0.1524" layer="16"/>
+<wire x1="6.096" y1="39.116" x2="2.54" y2="39.116" width="0.1524" layer="16"/>
+<wire x1="33.02" y1="63.5" x2="12.7" y2="63.5" width="0.1524" layer="16"/>
+<wire x1="12.7" y1="63.5" x2="7.62" y2="58.42" width="0.1524" layer="16"/>
 </signal>
 <signal name="N$6">
@@
 <wire x1="36.83" y1="51.22" x2="36.83" y2="46.99" width="0.1524" layer="1"/>
 <via x="36.83" y="46.99" extent="1-16" drill="0.35"/>
-<wire x1="36.83" y1="46.99" x2="34.29" y2="44.45" width="0.1524" layer="16"/>
 <via x="21.59" y="44.45" extent="1-16" drill="0.35"/>
 <wire x1="21.59" y1="44.45" x2="21.59" y2="45.72" width="0.1524" layer="1"/>
 <wire x1="21.59" y1="45.72" x2="22.5125" y2="46.6425" width="0.1524" layer="1"/>
 <wire x1="22.5125" y1="46.6425" x2="23.7825" y2="46.6425" width="0.1524" layer="1"/>
-<wire x1="34.29" y1="44.45" x2="21.59" y2="44.45" width="0.1524" layer="16"/>
+<wire x1="21.59" y1="44.45" x2="21.59" y2="41.91" width="0.1524" layer="16"/>
+<wire x1="21.59" y1="41.91" x2="22.86" y2="40.64" width="0.1524" layer="16"/>
+<wire x1="22.86" y1="40.64" x2="30.48" y2="40.64" width="0.1524" layer="16"/>
+<wire x1="30.48" y1="40.64" x2="36.83" y2="46.99" width="0.1524" layer="16"/>
 </signal>
 <signal name="OUTPUT">
@@
 <wire x1="50.8" y1="61.81" x2="41.91" y2="52.92" width="0.1524" layer="1"/>
 <wire x1="41.91" y1="52.92" x2="36.83" y2="52.92" width="0.1524" layer="1"/>
-<wire x1="36.83" y1="52.92" x2="29.365" y2="52.92" width="0.1524" layer="1"/>
-<wire x1="29.365" y1="52.92" x2="24.07" y2="47.625" width="0.1524" layer="1"/>
+<wire x1="24.07" y1="50.74" x2="24.07" y2="47.625" width="0.1524" layer="1"/>
+<wire x1="36.83" y1="52.92" x2="26.25" y2="52.92" width="0.1524" layer="1"/>
+<wire x1="26.25" y1="52.92" x2="24.07" y2="50.74" width="0.1524" layer="1"/>
 </signal>
 <signal name="N$1">
@@
 <contactref element="OP1" pad="6"/>
 <contactref element="IC1" pad="5"/>
-<wire x1="29.27" y1="46.355" x2="29.27" y2="45.9017125" width="0.1524" layer="1"/>
-<wire x1="29.27" y1="45.9017125" x2="29.27" y2="45.085" width="0.1524" layer="1"/>
+<wire x1="29.27" y1="46.355" x2="29.27" y2="45.085" width="0.1524" layer="1"/>
 <wire x1="24.07" y1="45.085" x2="29.27" y2="45.085" width="0.1524" layer="1"/>
 <wire x1="33.02" y1="55.88" x2="29.21" y2="52.07" width="0.1524" layer="16"/>
@@
 <via x="29.21" y="49.53" extent="1-16" drill="0.35"/>
 <wire x1="27.9414" y1="48.0196875" x2="27.9414" y2="47.2303125" width="0.1524" layer="1"/>
-<wire x1="27.9414" y1="47.2303125" x2="29.27" y2="45.9017125" width="0.1524" layer="1"/>
 <wire x1="29.21" y1="49.53" x2="29.21" y2="49.2882875" width="0.1524" layer="1"/>
 <wire x1="29.21" y1="49.2882875" x2="27.9414" y2="48.0196875" width="0.1524" layer="1"/>
+<wire x1="27.9414" y1="47.2303125" x2="28.8167125" y2="46.355" width="0.1524" layer="1"/>
+<wire x1="28.8167125" y1="46.355" x2="29.27" y2="46.355" width="0.1524" layer="1"/>
 </signal>
 <signal name="3.3V">
@@
 <contactref element="OP1" pad="8"/>
 <contactref element="CSAFE" pad="2"/>
-<wire x1="38.1" y1="55.88" x2="45.72" y2="48.26" width="0.1524" layer="16"/>
-<wire x1="50.8" y1="48.26" x2="45.72" y2="48.26" width="0.1524" layer="16"/>
 <wire x1="46.99" y1="49.95" x2="48.68" y2="48.26" width="0.1524" layer="1"/>
 <wire x1="48.68" y1="48.26" x2="50.8" y2="48.26" width="0.1524" layer="1"/>
@@
 <wire x1="31.75" y1="48.26" x2="31.115" y2="47.625" width="0.1524" layer="1"/>
 <wire x1="31.115" y1="47.625" x2="29.27" y2="47.625" width="0.1524" layer="1"/>
+<wire x1="38.1" y1="55.88" x2="38.1" y2="49.53" width="0.1524" layer="16"/>
+<wire x1="38.1" y1="49.53" x2="39.37" y2="48.26" width="0.1524" layer="16"/>
+<wire x1="39.37" y1="48.26" x2="50.8" y2="48.26" width="0.1524" layer="16"/>
 </signal>
 <signal name="N$3">
@@
 <contactref element="IC1" pad="6"/>
 <contactref element="RIN" pad="1"/>
-<wire x1="32.9048" y1="53.2248" x2="29.23874375" y2="53.2248" width="0.1524" layer="1"/>
-<wire x1="28.08394375" y1="52.07" x2="13.97" y2="52.07" width="0.1524" layer="1"/>
-<wire x1="29.23874375" y1="53.2248" x2="28.08394375" y2="52.07" width="0.1524" layer="1"/>
 <wire x1="13.97" y1="52.07" x2="12.7" y2="50.8" width="0.1524" layer="1"/>
 <wire x1="12.7" y1="50.8" x2="12.7" y2="43.18" width="0.1524" layer="1"/>
 <wire x1="12.7" y1="43.18" x2="13.97" y2="41.91" width="0.1524" layer="1"/>
-<wire x1="35.56" y1="55.88" x2="32.9048" y2="53.2248" width="0.1524" layer="1"/>
 <wire x1="13.97" y1="41.91" x2="14.82" y2="41.91" width="0.1524" layer="1"/>
 <wire x1="14.82" y1="41.91" x2="17.36" y2="44.45" width="0.1524" layer="1"/>
+<wire x1="35.56" y1="55.88" x2="35.56" y2="54.61" width="0.1524" layer="1"/>
+<wire x1="24.13" y1="54.61" x2="21.59" y2="52.07" width="0.1524" layer="1"/>
+<wire x1="21.59" y1="52.07" x2="13.97" y2="52.07" width="0.1524" layer="1"/>
+<wire x1="35.56" y1="54.61" x2="24.13" y2="54.61" width="0.1524" layer="1"/>
 </signal>
 <signal name="N$5">
 <contactref element="R3" pad="1"/>
 <contactref element="IC1" pad="1"/>
-<wire x1="40.64" y1="63.5" x2="42.76" y2="63.5" width="0.1524" layer="1"/>
-<wire x1="42.76" y1="63.5" x2="45.72" y2="60.54" width="0.1524" layer="1"/>
+<wire x1="40.64" y1="63.5" x2="41.49" y2="63.5" width="0.1524" layer="1"/>
+<wire x1="41.49" y1="63.5" x2="44.45" y2="60.54" width="0.1524" layer="1"/>
 </signal>
 <signal name="N$7">
 <contactref element="R3" pad="2"/>
 <contactref element="IC1" pad="8"/>
-<wire x1="40.64" y1="55.88" x2="42.76" y2="55.88" width="0.1524" layer="1"/>
-<wire x1="42.76" y1="55.88" x2="45.72" y2="58.84" width="0.1524" layer="1"/>
+<wire x1="40.64" y1="55.88" x2="41.49" y2="55.88" width="0.1524" layer="1"/>
+<wire x1="41.49" y1="55.88" x2="44.45" y2="58.84" width="0.1524" layer="1"/>
 </signal>
 <signal name="N$8">
@@
 <wire x1="39.7922" y1="73.5222" x2="41.35" y2="75.08" width="0.1524" layer="1"/>
 <wire x1="39.7922" y1="71.9790625" x2="39.7922" y2="73.5222" width="0.1524" layer="1"/>
-<wire x1="35.56" y1="63.5" x2="35.56" y2="67.7468625" width="0.1524" layer="1"/>
-<wire x1="35.56" y1="67.7468625" x2="39.7922" y2="71.9790625" width="0.1524" layer="1"/>
+<wire x1="39.7922" y1="71.9790625" x2="35.56" y2="67.7468625" width="0.1524" layer="1"/>
+<wire x1="35.56" y1="67.7468625" x2="35.56" y2="63.5" width="0.1524" layer="1"/>
 </signal>
 </signals>

Commit message: Week7
Routing:
- net 3.3V: track 54.7 -> 53.8 mm
- net N$4: track 39.6 -> 38.8 mm
Changed lines of the file:
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@@
 <wire x1="46.99" y1="49.95" x2="48.68" y2="48.26" width="0.1524" layer="1"/>
 <wire x1="48.68" y1="48.26" x2="50.8" y2="48.26" width="0.1524" layer="1"/>
-<wire x1="22.86" y1="35.98" x2="24.55" y2="35.98" width="0.1524" layer="1"/>
-<wire x1="24.55" y1="35.98" x2="33.02" y2="44.45" width="0.1524" layer="1"/>
-<wire x1="33.02" y1="44.45" x2="33.02" y2="45.72" width="0.1524" layer="1"/>
-<wire x1="33.02" y1="45.72" x2="31.115" y2="47.625" width="0.1524" layer="1"/>
+<wire x1="22.86" y1="35.98" x2="24.13" y2="35.98" width="0.1524" layer="1"/>
 <wire x1="38.1" y1="55.88" x2="31.75" y2="49.53" width="0.1524" layer="16"/>
 <wire x1="31.75" y1="49.53" x2="31.75" y2="48.26" width="0.1524" layer="16"/>
@@
 <wire x1="38.1" y1="49.53" x2="39.37" y2="48.26" width="0.1524" layer="16"/>
 <wire x1="39.37" y1="48.26" x2="50.8" y2="48.26" width="0.1524" layer="16"/>
+<wire x1="31.75" y1="48.26" x2="31.75" y2="43.6" width="0.1524" layer="1"/>
+<wire x1="31.75" y1="43.6" x2="24.13" y2="35.98" width="0.1524" layer="1"/>
 </signal>
 <signal name="N$3">
@@
 <contactref element="IC1" pad="6"/>
 <contactref element="RIN" pad="1"/>
-<wire x1="13.97" y1="52.07" x2="12.7" y2="50.8" width="0.1524" layer="1"/>
+<wire x1="12.7" y1="50.8" x2="13.97" y2="52.07" width="0.1524" layer="1"/>
 <wire x1="12.7" y1="50.8" x2="12.7" y2="43.18" width="0.1524" layer="1"/>
 <wire x1="12.7" y1="43.18" x2="13.97" y2="41.91" width="0.1524" layer="1"/>
 <wire x1="13.97" y1="41.91" x2="14.82" y2="41.91" width="0.1524" layer="1"/>
 <wire x1="14.82" y1="41.91" x2="17.36" y2="44.45" width="0.1524" layer="1"/>
-<wire x1="35.56" y1="55.88" x2="35.56" y2="54.61" width="0.1524" layer="1"/>
 <wire x1="24.13" y1="54.61" x2="21.59" y2="52.07" width="0.1524" layer="1"/>
-<wire x1="21.59" y1="52.07" x2="13.97" y2="52.07" width="0.1524" layer="1"/>
-<wire x1="35.56" y1="54.61" x2="24.13" y2="54.61" width="0.1524" layer="1"/>
+<wire x1="13.97" y1="52.07" x2="21.59" y2="52.07" width="0.1524" layer="1"/>
+<wire x1="35.56" y1="55.88" x2="34.29" y2="54.61" width="0.1524" layer="1"/>
+<wire x1="34.29" y1="54.61" x2="24.13" y2="54.61" width="0.1524" layer="1"/>
 </signal>
 <signal name="N$5">
