File: Hardware/Curios.brd (EAGLE design)
At the start: 53.3 x 59.7 mm, 13 parts, among them IC1 AD623N

Commit message: Week7
Routing:
- net GND: track 137.5 -> 13.4 mm, vias 0 -> 5
- net 3.3V: track 53.8 -> 0.00 mm, vias 1 -> 0
Changed lines of the file:
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@@
 <contactref element="J1" pad="GND"/>
 <contactref element="CSAFE" pad="1"/>
-<wire x1="33.02" y1="63.5" x2="33.02" y2="68.15" width="0.1524" layer="1"/>
-<wire x1="33.02" y1="68.15" x2="34.85" y2="69.98" width="0.1524" layer="1"/>
-<wire x1="34.85" y1="69.98" x2="36.4078" y2="71.5378" width="0.1524" layer="1"/>
-<wire x1="36.4078" y1="71.5378" x2="36.4078" y2="75.5946625" width="0.1524" layer="1"/>
-<wire x1="36.4078" y1="75.5946625" x2="39.46156875" y2="78.64843125" width="0.1524" layer="1"/>
-<wire x1="39.46156875" y1="78.64843125" x2="40.78156875" y2="78.64843125" width="0.1524" layer="1"/>
-<wire x1="40.78156875" y1="78.64843125" x2="41.35" y2="78.08" width="0.1524" layer="1"/>
-<wire x1="27.9900125" y1="78.88000625" x2="31.60999375" y2="78.88000625" width="0.1524" layer="1"/>
-<wire x1="34.85" y1="75.64" x2="34.85" y2="69.98" width="0.1524" layer="1"/>
-<wire x1="31.60999375" y1="78.88000625" x2="34.85" y2="75.64" width="0.1524" layer="1"/>
-<wire x1="50.8" y1="55.88" x2="50.8" y2="53.34" width="0.1524" layer="16"/>
-<wire x1="46.99" y1="51.65" x2="48.68" y2="53.34" width="0.1524" layer="1"/>
-<wire x1="48.68" y1="53.34" x2="50.8" y2="53.34" width="0.1524" layer="1"/>
-<wire x1="24.07" y1="43.815" x2="19.205" y2="38.95" width="0.1524" layer="1"/>
-<wire x1="19.205" y1="38.95" x2="15.24" y2="38.95" width="0.1524" layer="1"/>
-<wire x1="2.54" y1="39.116" x2="15.074" y2="39.116" width="0.1524" layer="1"/>
 <wire x1="15.074" y1="39.116" x2="15.24" y2="38.95" width="0.1524" layer="1"/>
-<wire x1="41.91" y1="64.77" x2="34.29" y2="64.77" width="0.1524" layer="16"/>
-<wire x1="34.29" y1="64.77" x2="33.02" y2="63.5" width="0.1524" layer="16"/>
-<wire x1="50.8" y1="55.88" x2="41.91" y2="64.77" width="0.1524" layer="16"/>
-<wire x1="7.62" y1="58.42" x2="7.62" y2="40.64" width="0.1524" layer="16"/>
-<wire x1="7.62" y1="40.64" x2="6.096" y2="39.116" width="0.1524" layer="16"/>
-<wire x1="6.096" y1="39.116" x2="2.54" y2="39.116" width="0.1524" layer="16"/>
-<wire x1="33.02" y1="63.5" x2="12.7" y2="63.5" width="0.1524" layer="16"/>
-<wire x1="12.7" y1="63.5" x2="7.62" y2="58.42" width="0.1524" layer="16"/>
 <polygon width="0.2032" layer="16" isolate="0.254">
-<vertex x="1.27" y="77.47"/>
+<vertex x="1.27" y="80.01"/>
 <vertex x="1.27" y="27.94"/>
 <vertex x="52.07" y="27.94"/>
-<vertex x="52.07" y="77.47"/>
+<vertex x="52.07" y="80.01"/>
 </polygon>
+<wire x1="24.07" y1="43.815" x2="24.13" y2="41.91" width="0.2032" layer="1"/>
+<wire x1="15.24" y1="38.95" x2="16.51" y2="40.64" width="0.2032" layer="1"/>
+<via x="16.51" y="40.64" extent="1-16" drill="0.35"/>
+<via x="24.13" y="41.91" extent="1-16" drill="0.35"/>
+<wire x1="46.99" y1="51.65" x2="45.72" y2="53.34" width="0.2032" layer="1"/>
+<via x="45.72" y="53.34" extent="1-16" drill="0.35"/>
+<wire x1="41.35" y1="78.08" x2="44.45" y2="76.2" width="0.2032" layer="1"/>
+<wire x1="34.85" y1="69.98" x2="31.75" y2="68.58" width="0.2032" layer="1"/>
+<via x="31.75" y="68.58" extent="1-16" drill="0.35"/>
+<via x="44.45" y="76.2" extent="1-16" drill="0.35"/>
 </signal>
 <signal name="N$6">
@@
 <contactref element="OP1" pad="8"/>
 <contactref element="CSAFE" pad="2"/>
-<wire x1="46.99" y1="49.95" x2="48.68" y2="48.26" width="0.1524" layer="1"/>
-<wire x1="48.68" y1="48.26" x2="50.8" y2="48.26" width="0.1524" layer="1"/>
-<wire x1="22.86" y1="35.98" x2="24.13" y2="35.98" width="0.1524" layer="1"/>
-<wire x1="38.1" y1="55.88" x2="31.75" y2="49.53" width="0.1524" layer="16"/>
-<wire x1="31.75" y1="49.53" x2="31.75" y2="48.26" width="0.1524" layer="16"/>
-<via x="31.75" y="48.26" extent="1-16" drill="0.35"/>
-<wire x1="31.75" y1="48.26" x2="31.115" y2="47.625" width="0.1524" layer="1"/>
-<wire x1="31.115" y1="47.625" x2="29.27" y2="47.625" width="0.1524" layer="1"/>
-<wire x1="38.1" y1="55.88" x2="38.1" y2="49.53" width="0.1524" layer="16"/>
-<wire x1="38.1" y1="49.53" x2="39.37" y2="48.26" width="0.1524" layer="16"/>
-<wire x1="39.37" y1="48.26" x2="50.8" y2="48.26" width="0.1524" layer="16"/>
-<wire x1="31.75" y1="48.26" x2="31.75" y2="43.6" width="0.1524" layer="1"/>
-<wire x1="31.75" y1="43.6" x2="24.13" y2="35.98" width="0.1524" layer="1"/>
 <polygon width="0.2032" layer="1" isolate="0.254">
 <vertex x="3.81" y="77.47"/>
